File: keyboards/rtenerowicz/rev1/pcbs/left/v1/left.kicad_pcb (KiCad board)
At the start: 2 copper layers, 143.8 x 104.1 mm, 72 parts

Commit message: pcb rev2
Parts:
- moved ? 0.60 mm to (272.8, 144.0)
Connections:
- ? pad 13: B6 -> VCC
Routing:
- net GND: track 187.6 -> 158.6 mm, vias 2 -> 3
- net VCC: track 163.6 -> 139.4 mm, vias 1 -> 2
- net D5: track 101.5 -> 118.7 mm, vias 2 -> 7
- net D1: track 32.8 -> 42.1 mm, vias 2 -> 5
- net D7: track 149.2 -> 154.3 mm
- net mr_diode: track 109.4 -> 112.4 mm
- net D0: track 43.0 -> 44.4 mm
- net B7: track 251.1 -> 252.4 mm
- net trackpoint_reset: track 93.1 -> 94.2 mm
- net C6: track 129.4 -> 130.4 mm
- net C7: track 196.1 -> 195.4 mm
- net E6: track 194.4 -> 194.9 mm
